Commit message: rviz works now

File: src/mini_bot_description/urdf/gazebo_control.xacro (robot description, xacro)
@@ -2,5 +2,5 @@
 <robot xmlns:xacro="http://www.ros.org/wiki/xacro">
     <gazebo>
-        <plugin name="diff_drive" filename="libgazebo_ros_diff_drive.so">
+        <plugin name="gz::sim::systems::DiffDrive" filename="gz-sim-diff-drive-system">
             <!-- Wheel Information -->
             <left_joint>left_wheel_joint</left_joint>

File: src/mini_bot_description/urdf/robot_core.xacro (robot description, xacro)
@@ -1,5 +1,5 @@
 <?xml version="1.0"?>
 <robot xmlns:xacro="http://www.ros.org/wiki/xacro">
-  <xacro:include filename="inertial_ macros.xacro"/>
+  <xacro:include filename="inertial_macros.xacro"/>
   <material name="white">
     <color rgba= "1 1 1 1" />
@@ -21,5 +21,5 @@
     <parent link= "base_link"/>
     <child link= "chassis"/>
-    <origin xyz="0.1 0 0"/>
+    <origin xyz="-0.1 0 0"/>
   </joint>
   <link name= "chassis">
@@ -54,5 +54,5 @@
     <visual>
       <geometry>
-        <cylinder radius="0.05" length="0.04"/>
+        <cylinder radius="0.07" length="0.04"/>
       </geometry>
       <material name="blue"/>
@@ -60,5 +60,5 @@
     <collision>
       <geometry>
-        <cylinder radius="0.05" length="0.04"/>
+        <cylinder radius="0.07" length="0.04"/>
       </geometry>
     </collision>
@@ -80,5 +80,5 @@
     <visual>
       <geometry>
-        <cylinder radius="0.05" length="0.04"/>
+        <cylinder radius="0.07" length="0.04"/>
       </geometry>
       <material name="blue"/>
@@ -86,5 +86,5 @@
     <collision>
       <geometry>
-        <cylinder radius="0.05" length="0.04"/>
+        <cylinder radius="0.07" length="0.04"/>
       </geometry>
     </collision>
@@ -100,4 +100,5 @@
     <parent link="chassis"/>
     <child link="caster_wheel"/>
+    <origin xyz="0.24 0 0"/>
   </joint>
   <link name="caster_wheel">

Commit message: changed robot structure

File: src/mini_bot_description/urdf/gazebo_control.xacro (robot description, xacro)
@@ -4,6 +4,8 @@
         <plugin name="gz::sim::systems::DiffDrive" filename="gz-sim-diff-drive-system">
             <!-- Wheel Information -->
-            <left_joint>left_wheel_joint</left_joint>
-            <right_joint>right_wheel_joint</right_joint>
+            <left_joint>front_left_wheel_joint</left_joint>
+            <left_joint>rear_left_wheel_joint</left_joint>
+            <right_joint>front_right_wheel_joint</right_joint>
+            <right_joint>rear_right_wheel_joint</right_joint>
             <wheel_separation>0.297</wheel_separation>
             <wheel_diameter>0.066</wheel_diameter>

File: src/mini_bot_description/urdf/robot_core.xacro (robot description, xacro)
@@ -25,18 +25,18 @@
   <link name= "chassis">
     <visual>
-      <origin xyz="0.15 0 0.075"/>
+      <origin xyz="0.15 0 0.072"/>
       <geometry>
-        <box size="0.3 0.3 0.15"/>
+        <box size="0.35 0.3 0.15"/>
       </geometry>
       <material name="white" />
     </visual>
      <collision>
-      <origin xyz="0.15 0 0.075"/>
+      <origin xyz="0.15 0 0.072"/>
       <geometry>
-        <box size="0.3 0.3 0.15"/>
+        <box size="0.35 0.3 0.15"/>
       </geometry>
     </collision>
     <xacro:inertial_box mass="0.5" x="0.3" y="0.3" z="0.15">
-      <origin xyz="0.15 0 0.075" rpy="0 0 0"/>
+      <origin xyz="0.15 0 0.072" rpy="0 0 0"/>
     </xacro:inertial_box>
   </link>
@@ -44,12 +44,12 @@
     <material>Gazebo/White</material>
   </gazebo>
-  <!--LEFT WHEEL LINK-->
-  <joint name="left_wheel_joint" type="continuous">
+  <!--FRONT LEFT WHEEL LINK-->
+  <joint name="front_left_wheel_joint" type="continuous">
     <parent link="base_link"/>
-    <child link="left_wheel"/>
-    <origin xyz="0 0.175 0" rpy="-${pi/2} 0 0"/>
+    <child link="front_left_wheel"/>
+    <origin xyz="0.15 0.175 0" rpy="-${pi/2} 0 0"/>
     <axis xyz="0 0 1"/>
   </joint>
-  <link name="left_wheel">
+  <link name="front_left_wheel">
     <visual>
       <geometry>
@@ -67,15 +67,15 @@
     </xacro:inertial_cylinder>
   </link>
-  <gazebo reference="left_wheel">
+  <gazebo reference="front_left_wheel">
     <material>Gazebo/Blue</material>
   </gazebo>
-  <!--RIGHT WHEEL LINK-->
-  <joint name="right_wheel_joint" type="continuous">
+  <!--FRONT RIGHT WHEEL LINK-->
+  <joint name="front_right_wheel_joint" type="continuous">
     <parent link="base_link"/>
-    <child link="right_wheel"/>
-    <origin xyz="0 -0.175 0" rpy="${pi/2} 0 0"/>
+    <child link="front_right_wheel"/>
+    <origin xyz="0.15 -0.175 0" rpy="${pi/2} 0 0"/>
     <axis xyz="0 0 -1"/>
   </joint>
-  <link name="right_wheel">
+  <link name="front_right_wheel">
     <visual>
       <geometry>
@@ -93,33 +93,58 @@
     </xacro:inertial_cylinder>
   </link>
-  <gazebo reference="right_wheel">
+  <gazebo reference="front_right_wheel">
     <material>Gazebo/Blue</material>
   </gazebo>
-  <!--CASTER WHEEL LINK-->
-  <joint name="caster_wheel_joint" type="fixed">
-    <parent link="chassis"/>
-    <child link="caster_wheel"/>
-    <origin xyz="0.24 0 0"/>
+  <!--REAR LEFT WHEEL LINK-->
+  <joint name="rear_left_wheel_joint" type="continuous">
+    <parent link="base_link"/>
+    <child link="rear_left_wheel"/>
+    <origin xyz="-0.1 0.175 0" rpy="-${pi/2} 0 0"/>
+    <axis xyz="0 0 1"/>
   </joint>
-  <link name="caster_wheel">
+  <link name="rear_left_wheel">
     <visual>
       <geometry>
-        <sphere radius="0.05"/>
+        <cylinder radius="0.07" length="0.04"/>
       </geometry>
-      <material name="black"/>
+      <material name="blue"/>
     </visual>
     <collision>
       <geometry>
-        <sphere radius="0.05"/>
+        <cylinder radius="0.07" length="0.04"/>
       </geometry>
     </collision>
-    <xacro:inertial_sphere mass="0.1" radius="0.05">
-        <origin xyz="0 0 0" rpy="0 0 0"/>
-    </xacro:inertial_sphere>
+    <xacro:inertial_cylinder mass="0.1" length="0.04" radius="0.05">
+      <origin xyz="0 0 0" rpy="0 0 0"/>
+    </xacro:inertial_cylinder>
   </link>
-  <gazebo reference="caster_wheel">
-    <material>Gazebo/Black</material>
-    <mu1 value = "0.001"/>
-    <mu2 value = "0.001"/>
+  <gazebo reference="rear_left_wheel">
+    <material>Gazebo/Blue</material>
+  </gazebo>
+  <!--REAR RIGHT WHEEL LINK-->
+  <joint name="rear_right_wheel_joint" type="continuous">
+    <parent link="base_link"/>
+    <child link="rear_right_wheel"/>
+    <origin xyz="-0.1 -0.175 0" rpy="${pi/2} 0 0"/>
+    <axis xyz="0 0 -1"/>
+  </joint>
+  <link name="rear_right_wheel">
+    <visual>
+      <geometry>
+        <cylinder radius="0.07" length="0.04"/>
+      </geometry>
+      <material name="blue"/>
+    </visual>
+    <collision>
+      <geometry>
+        <cylinder radius="0.07" length="0.04"/>
+      </geometry>
+    </collision>
+    <xacro:inertial_cylinder mass="0.1" length="0.04" radius="0.05">
+      <origin xyz="0 0 0" rpy="0 0 0"/>
+    </xacro:inertial_cylinder>
+  </link>
+  <gazebo reference="rear_right_wheel">
+    <material>Gazebo/Blue</material>
   </gazebo>
 </robot>
